File: Transistor_Ladder_VCF/PCB/Transistor_Ladder_VCF.kicad_pcb (KiCad board)
At the start: 2 copper layers, 39.7 x 109.8 mm, 126 parts, among them J1 Audio-Jack-2_Switch, J2 Audio-Jack-2_Switch, J3 Audio-Jack-2_Switch, J4 Audio-Jack-2_Switch, J5 Audio-Jack-2_Switch, J6 Audio-Jack-2_Switch, J7 Audio-Jack-2_Switch, J8 Conn_02x05_Odd_Even, Q1 BCM847BS,135, Q2 BCM847BS,135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

Commit message: Updated some resistor values
Parts:
- R26: value 56k -> 100k
- RV3, RV6: value A100k -> B100k
- RV7, RV8: value B100k -> A100k
