File: Transistor_Ladder_VCF/PCB/Transistor_Ladder_VCF.kicad_pcb (KiCad board)
At the start: 2 copper layers, 39.7 x 109.8 mm, 126 parts, among them J1 Audio-Jack-2_Switch, J2 Audio-Jack-2_Switch, J3 Audio-Jack-2_Switch, J4 Audio-Jack-2_Switch, J5 Audio-Jack-2_Switch, J6 Audio-Jack-2_Switch, J7 Audio-Jack-2_Switch, J8 Conn_02x05_Odd_Even, Q1 BCM847BS,135, Q2 BCM847BS,135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

Commit message: Updated schematics and BOM
Parts:
- R43: value 2k2 -> 2k7
- RV12: value 10k -> 100k
