File: Transistor_Ladder_VCF/PCB/Transistor_Ladder_VCF.sch (KiCad schematic (older format))
At the start: 126 parts, among them J1 Audio-Jack-2_Switch, J2 Audio-Jack-2_Switch, J3 Audio-Jack-2_Switch, J4 Audio-Jack-2_Switch, J5 Audio-Jack-2_Switch, J6 Audio-Jack-2_Switch, J7 Audio-Jack-2_Switch, J8 Conn_02x05_Odd_Even, Q1 BCM847BS,135, Q2 BCM847BS,135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

Commit message: Updated schematics and BOM
Parts:
- R43: value 2k2 -> 2k7
- RV12: value 10k -> 100k
Changed lines of the file:
@@
 P 7700 5950
 F 0 "RV12" V 7525 5950 50  0000 C CNN
-F 1 "10k" V 7600 5950 50  0000 C CNN
+F 1 "100k" V 7600 5950 50  0000 C CNN
 F 2 "Eigenes:Trim_pot" H 7700 5950 50  0001 C CNN
 F 3 "" H 7700 5950 50  0001 C CNN
@@
 P 7300 4250
 F 0 "R43" V 7380 4250 50  0000 C CNN
-F 1 "2k2" V 7300 4250 50  0000 C CNN
+F 1 "2k7" V 7300 4250 50  0000 C CNN
 F 2 "Resistor_SMD:R_0603_1608Metric_Pad0.98x0.95mm_HandSolder" V 7230 4250 50  0001 C CNN
 F 3 "" H 7300 4250 50  0001 C CNN
