File: Betula/Betula_ADAT/Betula_ADAT.kicad_pcb (KiCad board)
At the start: 2 copper layers, 39.5 x 12.8 mm, 6 parts, among them J1 Optical_Transmitter, J2 Optical_Receiver, J3 Conn_02x02_Top_Bottom

Commit message: Incremented all version numbers to 1.5.1 on all PCBs
Other:
- board text added: "Blattwerk Betula V1.5.1 ADAT In/Out"
- board text removed: "Blattwerk Betula V1.4 ADAT In/Out"
Changed lines of the file:
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@@
 		)
 	)
-	(gr_text "Blattwerk Betula V1.4 ADAT In/Out"
-		(at 117.72 64.92 0)
+	(gr_text "Blattwerk Betula V1.5.1 ADAT In/Out"
+		(at 117.983 64.77 0)
 		(layer "B.SilkS")
 		(effects
