File: Betula/Betula_Output/Betula_Output.kicad_pcb (KiCad board)
At the start: 2 copper layers, 39.4 x 43.2 mm, 77 parts, among them J1 AudioJack2_SwitchT, J2 AudioJack2_SwitchT, J3 AudioJack2_SwitchT, J4 AudioJack2_SwitchT, J5 AudioJack2_SwitchT, J6 AudioJack2_SwitchT, J7 AudioJack2_SwitchT, J8 AudioJack2_SwitchT, J9 Conn_02x15_Top_Bottom, U1 OPA1692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

Commit message: Incremented all version numbers to 1.5.1 on all PCBs
Other:
- board text added: "BETULA OUTPUT V1.5.1"
- board text removed: "BETULA OUTPUT V1.4"
Changed lines of the file:
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@@
 		(layer "Edge.Cuts")
 	)
-	(gr_text "BETULA       OUTPUT         V1.4\n\n"
-		(at 139.76 91.82 0)
+	(gr_text "BETULA     OUTPUT      V1.5.1\n\n"
+		(at 139.7 91.82 0)
 		(layer "B.SilkS")
 		(effects
